File: cpu-z80.sch (KiCad schematic (older format))
At the start: 19 parts, among them Q6 2SC1815, U10 Z80, U12 74LS373, U13 74LS244, U31 74LS00, U37 7406, U56 74LS74, U60 7407, U8 74LS08

Commit message: Fix R47/R101
Parts:
- renumbered R47 to R101
Changed lines of the file:
@@
 $EndComp
 $Comp
-L Device:R R47
+L Device:R R101
 U 1 1 5E03F3BC
 P 2200 2400
-F 0 "R47" V 2100 2400 50  0000 C CNN
+F 0 "R101" V 2100 2400 50  0000 C CNN
 F 1 "1k" V 2200 2400 39  0000 C CNN
 F 2 "Open128:R_Axial_DIN0309_L9.0mm_D2.5mm_P12.70mm_Horizontal" V 2130 2400 50  0001 C CNN

Commit message: Clean up schematic
Connections:
- net Z80_RW renamed Z80_R~W
- net ~Z80IO renamed ~Z80_IO
Changed lines of the file:
@@
 Wire Wire Line
 	4000 2500 4400 2500
-Text HLabel 4000 3200 0    50   Input ~ 0
-~IRQ
 Wire Wire Line
 	4000 3200 4400 3200
-Text HLabel 4000 3500 0    50   Output ~ 0
-~M1
 Wire Wire Line
 	4000 3500 4400 3500
@@
 	1    0    0    -1
 $EndComp
-Text HLabel 10600 900  2    50   Input ~ 0
-D1MHZ
 Wire Wire Line
 	8850 2950 9250 2950
@@
 Wire Wire Line
 	8350 3350 8350 3400
-Text HLabel 5000 6350 0    50   Input ~ 0
-GAEC
 Wire Wire Line
 	5000 6350 5500 6350
@@
 Wire Wire Line
 	6250 6250 7650 6250
-Text HLabel 6450 6750 2    50   Output ~ 0
-Z80_RW
-Text HLabel 4000 4900 0    50   Output ~ 0
-~BUSACK
 Wire Wire Line
 	4000 4900 4400 4900
@@
 	1    0    0    -1
 $EndComp
-Text HLabel 1150 5950 0    50   3State ~ 0
-~Z80IO
 $Comp
 L 74xx:74LS06 U37
@@
 Wire Wire Line
 	3000 3750 3000 3850
-Text HLabel 1150 5100 0    50   Input ~ 0
-~PLA_Z80EN
-Text HLabel 1150 5300 0    50   Input ~ 0
-~AEC
 Wire Wire Line
 	1150 5300 1250 5300
 Wire Wire Line
 	1150 5100 1250 5100
-Text HLabel 1150 4350 0    50   Input ~ 0
-BA
 Wire Wire Line
 	1150 4350 1900 4350
-Text HLabel 1150 4800 0    50   Input ~ 0
-~MMU_Z80EN
 Wire Wire Line
 	1150 4800 1900 4800
@@
 	1    0    0    -1
 $EndComp
-Text HLabel 1100 2200 0    50   Input ~ 0
-ΦZ80
 Wire Wire Line
 	1100 2200 1200 2200
@@
 Wire Bus Line
 	9150 1100 9150 4800
+Text GLabel 1150 4350 0    50   Input ~ 0
+BA
+Text GLabel 4000 3200 0    50   Input ~ 0
+~IRQ
+Text GLabel 1150 5300 0    50   Input ~ 0
+~AEC
+Text GLabel 10600 900  2    50   Input ~ 0
+D1MHZ
+Text GLabel 1100 2200 0    50   Input ~ 0
+ΦZ80
+Text GLabel 4000 3500 0    50   Output ~ 0
+~M1
+Text GLabel 4000 4900 0    50   Output ~ 0
+~BUSACK
+Text GLabel 1150 5950 0    50   3State ~ 0
+~Z80_IO
+Text GLabel 5000 6350 0    50   Input ~ 0
+GAEC
+Text GLabel 6450 6750 2    50   Output ~ 0
+Z80_R~W
+Text GLabel 1150 5100 0    50   Input ~ 0
+~PLA_Z80EN
+Text GLabel 1150 4800 0    50   Input ~ 0
+~MMU_Z80EN
 $EndSCHEMATC
