File: serialbus.sch (KiCad schematic (older format))
At the start: 25 parts, among them CN6 DIN6 Male, CN7 7 pin post, U16 74LS14, U30 7406, U37 7406, U58 74LS03, U60 7407, U8 74LS08

Commit message: Clean up schematic
Changed lines of the file:
@@
 	3250 2000 3400 2000
 NoConn ~ 5000 1350
-Text HLabel 4500 1500 0    50   Input ~ 0
-~DRESET
 Text HLabel 4800 3750 0    50   Input ~ 0
 ~EXTRES
@@
 Wire Wire Line
 	9150 3100 10600 3100
-Text HLabel 10600 3100 2    50   Input ~ 0
-128_64
 $Comp
 L 74xx:74LS14 U16
@@
 Wire Wire Line
 	9900 2900 10250 2900
-Text HLabel 10600 2900 2    50   Input ~ 0
-~FSDIR
 Wire Wire Line
 	8050 4900 10250 4900
@@
 Wire Wire Line
 	4750 4750 4750 4800
+Text GLabel 4500 1500 0    50   Input ~ 0
+~DRESET
+Text GLabel 10600 2900 2    50   Input ~ 0
+~FSDIR
+Text GLabel 10600 3100 2    50   Input ~ 0
+128_64
 $EndSCHEMATC
